File: 16n-midijack.brd (EAGLE design)
At the start: 248.9 x 101.6 mm, 21 parts

Commit message: SPI and MIDI breakouts.
Parts:
- added II: (no value), pinhead:1X04/90
- added R3, R4: (no value), rcl:R0805
- R1, R2: device SparkFun-Resistors:1206 -> rcl:R0805
- moved JP1 198.3 mm to (245.0, 15.0), turned to 180 degrees
- moved R2 168.4 mm to (230.0, 12.0), turned to 90 degrees
- moved S1 161.2 mm to (226.0, 3.17)
- moved R1 153.7 mm to (222.0, 12.0), turned to 90 degrees
Connections:
- new net SCL: II.3, R4.1, U$1.19/A5
- new net SDA: II.2, R3.1, U$1.18/A4
- net +3V3: now also II.1, R3.2, R4.2
- net A4: no longer U$1.18/A4
- net A5: no longer U$1.19/A5
- net GND: now also II.4
Routing:
- net MIDI_OUT: track 28.9 -> 197.2 mm, vias 0 -> 1
- net +5V: track 66.8 -> 226.0 mm
- net SDA: track 0.00 -> 48.4 mm
- net SCL: track 0.00 -> 46.7 mm
- net +3V3: track 379.0 -> 415.1 mm
- net N$1: track 15.1 -> 28.5 mm
- net A5: track 183.1 -> 174.2 mm
- net N$2: track 26.8 -> 21.0 mm
- net N$3: track 11.2 -> 15.1 mm
- net A4: track 194.3 -> 190.5 mm
- net N$4: track 13.6 -> 14.6 mm
Other:
- board text added: "3V3"
- board text added: "GND"
- board text added: "SCL"
- board text added: "SDA"

Commit message: Various changes:
- through hole componentry
- up-to-date silking
- protection diodes on II lines
Parts:
- added D1, D2, D3, D4: (no value), SparkFun-DiscreteSemi:DIODE-1N4148
- R1, R2: value 220R -> (none); device rcl:R0805 -> SparkFun-Resistors:AXIAL-0.3-KIT
- R3, R4: value (none) -> 4K7; device rcl:R0805 -> SparkFun-Resistors:AXIAL-0.3-KIT
- moved R4 25.9 mm to (73.7, 16.5)
- moved R3 10.8 mm to (62.2, 16.5)
- moved R2 7.89 mm to (223.5, 16.5)
- moved R1 5.06 mm to (219.7, 16.5)
- moved S1 2.54 mm to (226.1, 5.71)
- moved II 1.31 mm to (50.2, 7.30)
Connections:
- net +3V3: now also D2.C, D4.C, R3.P$2, R4.P$2; no longer II.1, R3.2, R4.2
- net +5V: now also II.1, R1.P$2; no longer R1.2
- net GND: now also D1.A, D3.A
- net MIDI_OUT: now also R2.P$2; no longer R2.2
- net N$3: now also R2.P$1; no longer R2.1
- net N$4: now also R1.P$1; no longer R1.1
- net SCL: now also D3.C, D4.A, R4.P$1; no longer R4.1
- net SDA: now also D1.C, D2.A, R3.P$1; no longer R3.1
Routing:
- net SCL: track 46.7 -> 80.3 mm
- net SDA: track 48.4 -> 66.1 mm
- net +3V3: track 415.1 -> 430.6 mm
- net N$3: track 15.1 -> 11.0 mm
- net MIDI_OUT: track 197.2 -> 193.7 mm, vias 1 -> 0
- net N$1: track 28.5 -> 26.0 mm
- net +5V: track 226.0 -> 226.7 mm
- net N$4: track 14.6 -> 15.3 mm
Other:
- board text added: "16"
- board text added: "220R"
- board text added: "4.7K, 1N4148"
- board text added: "5V"
- board text added: "Tip is +5V Ring is Out"
- board text removed: "3V3"
- board text removed: "Tip is +5V Ring is OUT"

Commit message: What I sent to Sean.
Connections:
- net MIDI_OUT: now also U$1.10; no longer U$1.12
Routing:
- net MIDI_OUT: track 193.7 -> 201.7 mm
Changed lines of the file:
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@@
 <setting verticaltext="up"/>
 </settings>
-<grid distance="12.5" unitdist="mil" unit="mil" style="lines" multiple="4" display="yes" altdistance="25" altunitdist="mil" altunit="mil"/>
+<grid distance="50" unitdist="mil" unit="mil" style="lines" multiple="1" display="no" altdistance="10" altunitdist="mil" altunit="mil"/>
 <layers>
 <layer number="1" name="Top" color="4" fill="1" visible="yes" active="yes"/>
@@
 <layer number="230" name="230bmp" color="7" fill="1" visible="no" active="yes"/>
 <layer number="231" name="231bmp" color="7" fill="1" visible="no" active="yes"/>
+<layer number="232" name="Eagle3D_PG2" color="7" fill="1" visible="no" active="no"/>
+<layer number="233" name="Eagle3D_PG3" color="7" fill="1" visible="no" active="no"/>
 <layer number="248" name="Housing" color="7" fill="1" visible="no" active="yes"/>
 <layer number="249" name="Edge" color="7" fill="1" visible="no" active="yes"/>
@@
 </signal>
 <signal name="MIDI_OUT">
-<contactref element="U$1" pad="12"/>
 <contactref element="R2" pad="P$2"/>
-<wire x1="35.56" y1="6.35" x2="209.55" y2="6.35" width="0.4064" layer="16"/>
-<wire x1="209.55" y1="6.35" x2="223.52" y2="20.32" width="0.4064" layer="16"/>
+<contactref element="U$1" pad="10"/>
+<wire x1="30.48" y1="6.35" x2="30.48" y2="5.08" width="0.4064" layer="1"/>
+<wire x1="30.48" y1="5.08" x2="31.75" y2="3.81" width="0.4064" layer="1"/>
+<wire x1="31.75" y1="3.81" x2="38.1" y2="3.81" width="0.4064" layer="1"/>
+<wire x1="38.1" y1="3.81" x2="40.64" y2="6.35" width="0.4064" layer="1"/>
+<wire x1="209.55" y1="6.35" x2="223.52" y2="20.32" width="0.4064" layer="1"/>
+<wire x1="40.64" y1="6.35" x2="209.55" y2="6.35" width="0.4064" layer="1"/>
 </signal>
 <signal name="N$1">

Commit message: Everything on the board.
Now needs routing. Oh boy.
Parts:
- added C1, C2, C3, C4, C5, C6, C7, C8: 100n, rcl:C0805
- added J1, J10, J11, J12, J13, J14, J15, J16, J2, J3, J4, J5, J6, J7, J8, J9: THONKICONNNEW, MusicThingModular:WQP-PJ301M-12_JACK
- added R10, R14, R15, R19, R20, R24, R25, R29, R30, R34, R35, R39, R40, R44, R5, R9: 5.6K, rcl:R0805
- added R11, R13, R16, R18, R21, R23, R26, R28, R31, R33, R36, R38, R41, R43, R6, R8: 10K, rcl:R0805
- added R12, R17, R22, R27, R32, R37, R42, R45, R46, R47, R48, R49, R50, R51, R52, R7: 100, rcl:R0805
- added U1, U2, U3, U4, U5, U6, U7, U8: MCP6004_SMD, MusicThingModular:SO14
- D1, D2, D3, D4: device SparkFun-DiscreteSemi:DIODE-1N4148 -> foxfield:SOD-123
- R1, R2: value (none) -> 220; device SparkFun-Resistors:AXIAL-0.3-KIT -> rcl:R0805
- R3, R4: device SparkFun-Resistors:AXIAL-0.3-KIT -> rcl:R0805
- moved D4 35.3 mm to (46.4, 21.6)
- moved R4 30.3 mm to (43.8, 21.6), turned to 270 degrees
- moved D3 29.0 mm to (48.9, 21.6)
- moved D2 16.7 mm to (54.0, 21.6)
- moved D1 15.5 mm to (51.4, 21.6)
- moved R1 9.69 mm to (228.0, 11.4)
- moved R3 7.65 mm to (56.5, 21.6), turned to 270 degrees
- moved R2 5.12 mm to (224.2, 11.4)
Connections:
- new net CV1: J1.P$1_TIP, R7.2
- new net CV10: J10.P$1_TIP, R48.2
- new net CV11: J11.P$1_TIP, R32.2
- new net CV12: J12.P$1_TIP, R49.2
- new net CV13: J13.P$1_TIP, R37.2
- new net CV14: J14.P$1_TIP, R50.2
- new net CV15: J15.P$1_TIP, R42.2
- new net CV16: J16.P$1_TIP, R51.2
- new net CV2: J2.P$1_TIP, R12.2
- new net CV3: J3.P$1_TIP, R52.2
- new net CV4: J4.P$1_TIP, R45.2
- new net CV5: J5.P$1_TIP, R17.2
- new net CV6: J6.P$1_TIP, R47.2
- new net CV7: J7.P$1_TIP, R22.2
- new net CV8: J8.P$1_TIP, R46.2
- new net CV9: J9.P$1_TIP, R27.2
- new net N$10: R8.2, R9.2, U1.12
- new net N$11: R17.1, U3.8, U3.9
- new net N$12: R15.2, R16.2, U3.10
- new net N$13: R18.2, R19.2, U3.12
- new net N$14: R22.1, U4.8, U4.9
- new net N$15: R20.2, R21.2, U4.10
- new net N$16: R23.2, R24.2, U4.12
- new net N$17: R27.1, U5.8, U5.9
- new net N$18: R25.2, R26.2, U5.10
- new net N$19: R28.2, R29.2, U5.12
- new net N$20: R32.1, U6.8, U6.9
- new net N$21: R30.2, R31.2, U6.10
- new net N$22: R33.2, R34.2, U6.12
- new net N$23: R37.1, U7.8, U7.9
- new net N$24: R35.2, R36.2, U7.10
- new net N$25: R38.2, R39.2, U7.12
- new net N$256: R12.1, U1.13, U1.14
- new net N$257: R45.1, U2.13, U2.14
- new net N$258: R47.1, U3.13, U3.14
- new net N$259: R46.1, U4.13, U4.14
- new net N$26: R42.1, U8.8, U8.9
- new net N$260: R48.1, U5.13, U5.14
- new net N$261: R49.1, U6.13, U6.14
- new net N$262: R50.1, U7.13, U7.14
- new net N$263: R51.1, U8.13, U8.14
- new net N$27: R40.2, R41.2, U8.10
- new net N$28: R43.2, R44.2, U8.12
- new net N$5: R52.1, U2.8, U2.9
- new net N$6: R10.2, R11.2, U2.10
- new net N$7: R13.2, R14.2, U2.12
- new net N$8: R7.1, U1.8, U1.9
- new net N$9: R5.2, R6.2, U1.10
- new net W0: R5.1, U$17.2, U1.5
- new net W1: R9.1, U$16.2, U1.3
- new net W10: R30.1, U$7.2, U6.5
- new net W11: R34.1, U$6.2, U6.3
- new net W12: R35.1, U$5.2, U7.5
- new net W13: R39.1, U$4.2, U7.3
- new net W14: R40.1, U$3.2, U8.5
- new net W15: R44.1, U$2.2, U8.3
- new net W2: R10.1, U$15.2, U2.5
- new net W3: R14.1, U$14.2, U2.3
- new net W4: R15.1, U$13.2, U3.5
- new net W5: R19.1, U$12.2, U3.3
- new net W6: R20.1, U$11.2, U4.5
- new net W7: R24.1, U$10.2, U4.3
- new net W8: R25.1, U$9.2, U5.5
- new net W9: R29.1, U$8.2, U5.3
- net +3V3: now also R3.2, R4.2; no longer R3.P$2, R4.P$2, U$10.1, U$11.1, U$12.1, U$13.1, U$14.1, U$15.1, U$16.1, U$17.1, U$2.1, U$3.1, U$4.1, U$5.1, U$6.1, U$7.1, U$8.1, U$9.1
- net +5V: now also C1.1, C2.1, C3.1, C4.1, C5.1, C6.1, C7.1, C8.1, R1.2, U$10.1, U$11.1, U$12.1, U$13.1, U$14.1, U$15.1, U$16.1, U$17.1, U$2.1, U$3.1, U$4.1, U$5.1, U$6.1, U$7.1, U$8.1, U$9.1, U1.4, U2.4, U3.4, U4.4, U5.4, U6.4, U7.4, U8.4; no longer R1.P$2
- net A0: now also U1.6, U1.7; no longer U$2.2
- net A1: now also U1.1, U1.2; no longer U$3.2
- net A10: now also U6.6, U6.7; no longer U$12.2
- net A11: now also U6.1, U6.2; no longer U$13.2
- net A12: now also U7.6, U7.7; no longer U$14.2
- net A13: now also U7.1, U7.2; no longer U$15.2
- net A14: now also U8.6, U8.7; no longer U$16.2
- net A15: now also U8.1, U8.2; no longer U$17.2
- net A2: now also U2.6, U2.7; no longer U$4.2
- net A3: now also U2.1, U2.2; no longer U$5.2
- net A4: now also U3.6, U3.7; no longer U$6.2
- net A5: now also U3.1, U3.2; no longer U$7.2
- net A6: now also U4.6, U4.7; no longer U$8.2
- net A7: now also U4.1, U4.2; no longer U$9.2
- net A8: now also U5.6, U5.7; no longer U$10.2
- net A9: now also U5.1, U5.2; no longer U$11.2
- net GND: now also C1.2, C2.2, C3.2, C4.2, C5.2, C6.2, C7.2, C8.2, J1.P$3_SLEEVE, J10.P$3_SLEEVE, J11.P$3_SLEEVE, J12.P$3_SLEEVE, J13.P$3_SLEEVE, J14.P$3_SLEEVE, J15.P$3_SLEEVE, J16.P$3_SLEEVE, J2.P$3_SLEEVE, J3.P$3_SLEEVE, J4.P$3_SLEEVE, J5.P$3_SLEEVE, J6.P$3_SLEEVE, J7.P$3_SLEEVE, J8.P$3_SLEEVE, J9.P$3_SLEEVE, R11.1, R13.1, R16.1, R18.1, R21.1, R23.1, R26.1, R28.1, R31.1, R33.1, R36.1, R38.1, R41.1, R43.1, R6.1, R8.1, U1.11, U2.11, U3.11, U4.11, U5.11, U6.11, U7.11, U8.11
- net MIDI_OUT: now also R2.2; no longer R2.P$2
- net N$3: now also R2.1; no longer R2.P$1
- net N$4: now also R1.1; no longer R1.P$1
- net SCL: now also R4.1; no longer R4.P$1
- net SDA: now also R3.1; no longer R3.P$1
Routing:
- net +5V: track 226.7 -> 822.4 mm, vias 0 -> 9
- net +3V3: track 430.6 -> 81.1 mm, vias 1 -> 0
- net A1: track 231.6 -> 1.27 mm
- net A2: track 218.2 -> 1.27 mm
- net A0: track 245.1 -> 32.3 mm, vias 0 -> 1
- net A3: track 204.7 -> 1.27 mm
- net A4: track 190.5 -> 1.27 mm
- net A6: track 174.8 -> 1.27 mm
- net A5: track 174.2 -> 1.27 mm
- net A7: track 161.4 -> 1.27 mm
- net A8: track 147.9 -> 1.27 mm
- net N$8: track 0.00 -> 143.5 mm, vias 0 -> 2
- net W0: track 0.00 -> 138.4 mm
- net A9: track 135.5 -> 1.27 mm
- net W1: track 0.00 -> 125.2 mm
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- added copper zone on layer 1, net GND
Other:
- board size 248.9 x 101.6 mm -> 248.9 x 120.7 mm
- board text removed: "220R"
- board text removed: "4.7K, 1N4148"

Commit message: Fixing up some layout.
Parts:
- moved R39 0.32 mm to (195.3, 19.1)
Routing:
- net W11: track 0.00 -> 14.5 mm
- net W7: track 0.00 -> 14.5 mm
- net W15: track 0.00 -> 14.5 mm
- net W5: track 0.00 -> 14.5 mm
- net W3: track 0.00 -> 14.5 mm
- net W13: track 0.00 -> 14.5 mm
- net W9: track 0.00 -> 14.5 mm
- net W8: track 0.00 -> 10.3 mm
- net W14: track 0.00 -> 10.3 mm
- net W12: track 0.00 -> 10.3 mm
- net W4: track 0.00 -> 10.3 mm
- net W10: track 0.00 -> 10.3 mm
- net W6: track 0.00 -> 10.1 mm
- net W2: track 0.00 -> 10.1 mm
- net N$21: track 0.00 -> 8.14 mm
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
Commit message: Boom. Routed.
Connections:
- net A4: now also U$1.18/A4
- net A5: now also U$1.19/A5
- net SCL: now also U$1.29; no longer U$1.19/A5
- net SDA: now also U$1.30; no longer U$1.18/A4
Routing:
- net A13: track 1.27 -> 222.6 mm, vias 0 -> 1
- net A12: track 1.27 -> 220.2 mm, vias 0 -> 1
- net A15: track 1.27 -> 209.3 mm, vias 0 -> 2
- net A14: track 1.27 -> 204.6 mm, vias 0 -> 2
- net A11: track 1.27 -> 184.4 mm, vias 0 -> 1
- net A10: track 1.27 -> 177.8 mm, vias 0 -> 1
- net A8: track 1.27 -> 147.7 mm, vias 0 -> 1
- net A9: track 1.27 -> 143.5 mm, vias 0 -> 1
- net N$5: track 1.27 -> 120.9 mm
- net A6: track 1.27 -> 120.5 mm, vias 0 -> 1
- net A7: track 1.27 -> 115.1 mm, vias 0 -> 1
- net N$11: track 1.27 -> 115.1 mm
- net N$263: track 1.27 -> 109.8 mm
- net W2: track 10.1 -> 117.0 mm
- net N$257: track 1.27 -> 107.2 mm
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Other:
- outline, holes or cut-outs redrawn

Commit message: New layout with horizontal jacks.
Parts:
- J1, J10, J11, J12, J13, J14, J15, J16, J2, J3, J4, J5, J6, J7, J8, J9: value THONKICONNNEW -> PJ302M; device MusicThingModular:WQP-PJ301M-12_JACK -> pj302m:PJ302M
- moved J1 6.67 mm to (10.2, 118.4), turned to 270 degrees
- moved J10 6.67 mm to (147.3, 118.4), turned to 270 degrees
- moved J11 6.67 mm to (162.6, 118.4), turned to 270 degrees
- moved J12 6.67 mm to (177.8, 118.4), turned to 270 degrees
- moved J13 6.67 mm to (193.0, 118.4), turned to 270 degrees
- moved J14 6.67 mm to (208.3, 118.4), turned to 270 degrees
- moved J15 6.67 mm to (223.5, 118.4), turned to 270 degrees
- moved J16 6.67 mm to (238.8, 118.4), turned to 270 degrees
- moved J2 6.67 mm to (25.4, 118.4), turned to 270 degrees
- moved J3 6.67 mm to (40.6, 118.4), turned to 270 degrees
- moved J4 6.67 mm to (55.9, 118.4), turned to 270 degrees
- moved J5 6.67 mm to (71.1, 118.4), turned to 270 degrees
- moved J6 6.67 mm to (86.4, 118.4), turned to 270 degrees
- moved J7 6.67 mm to (101.6, 118.4), turned to 270 degrees
- moved J8 6.67 mm to (116.8, 118.4), turned to 270 degrees
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Connections:
- net CV1: now also J1.TIP; no longer J1.P$1_TIP
- net CV10: now also J10.TIP; no longer J10.P$1_TIP
- net CV11: now also J11.TIP; no longer J11.P$1_TIP
- net CV12: now also J12.TIP; no longer J12.P$1_TIP
- net CV13: now also J13.TIP; no longer J13.P$1_TIP
- net CV14: now also J14.TIP; no longer J14.P$1_TIP
- net CV15: now also J15.TIP; no longer J15.P$1_TIP
- net CV16: now also J16.TIP; no longer J16.P$1_TIP
- net CV2: now also J2.TIP; no longer J2.P$1_TIP
- net CV3: now also J3.TIP; no longer J3.P$1_TIP
- net CV4: now also J4.TIP; no longer J4.P$1_TIP
- net CV5: now also J5.TIP; no longer J5.P$1_TIP
- net CV6: now also J6.TIP; no longer J6.P$1_TIP
- net CV7: now also J7.TIP; no longer J7.P$1_TIP
- net CV8: now also J8.TIP; no longer J8.P$1_TIP
- net CV9: now also J9.TIP; no longer J9.P$1_TIP
- net GND: now also J1.GND, J10.GND, J11.GND, J12.GND, J13.GND, J14.GND, J15.GND, J16.GND, J2.GND, J3.GND, J4.GND, J5.GND, J6.GND, J7.GND, J8.GND, J9.GND; no longer J1.P$3_SLEEVE, J10.P$3_SLEEVE, J11.P$3_SLEEVE, J12.P$3_SLEEVE, J13.P$3_SLEEVE, J14.P$3_SLEEVE, J15.P$3_SLEEVE, J16.P$3_SLEEVE, J2.P$3_SLEEVE, J3.P$3_SLEEVE, J4.P$3_SLEEVE, J5.P$3_SLEEVE, J6.P$3_SLEEVE, J7.P$3_SLEEVE, J8.P$3_SLEEVE, J9.P$3_SLEEVE
Routing:
- net CV16: track 16.7 -> 9.41 mm
- net CV5: track 16.9 -> 10.8 mm
- net CV10: track 16.9 -> 10.9 mm
- net CV13: track 16.7 -> 10.9 mm
- net CV4: track 16.7 -> 10.9 mm
- net CV3: track 16.7 -> 10.9 mm
- net CV6: track 16.7 -> 10.9 mm
- net CV11: track 16.7 -> 10.9 mm
- net CV2: track 16.7 -> 10.9 mm
- net CV1: track 16.7 -> 10.9 mm
- net CV7: track 16.5 -> 10.9 mm
- net CV8: track 16.7 -> 11.1 mm
- net CV14: track 16.7 -> 11.1 mm
- net CV9: track 16.7 -> 11.1 mm
- net CV15: track 16.7 -> 11.1 mm
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