File: 16n.brd (EAGLE design)
At the start: 248.9 x 120.7 mm, 110 parts, among them J1 PJ302M, J10 PJ302M, J11 PJ302M, J12 PJ302M, J13 PJ302M, J14 PJ302M, J15 PJ302M, J16 PJ302M, J2 PJ302M, J3 PJ302M, J4 PJ302M, J5 PJ302M, J6 PJ302M, J7 PJ302M, J8 PJ302M, J9 PJ302M, U1 MCP6004_SMD, U2 MCP6004_SMD, U3 MCP6004_SMD, U4 MCP6004_SMD, U5 MCP6004_SMD, U6 MCP6004_SMD, U7 MCP6004_SMD, U8 MCP6004_SMD

Commit message: V1.21: three support holes in the middle of the board. Drills 2.5.
Parts:
- moved FID1 0.57 mm to (2.54, 115.0)
Other:
- board text added: "v1.21"
- board text removed: "v1.2"
Changed lines of the file:
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@@
 <wire x1="0" y1="118.11" x2="0" y2="2.54" width="0" layer="20"/>
 <wire x1="0" y1="2.54" x2="2.54" y2="0" width="0" layer="20" curve="90"/>
-<hole x="2.54" y="2.54" drill="2"/>
-<hole x="246.38" y="99.06" drill="2"/>
-<hole x="246.38" y="2.54" drill="2"/>
-<hole x="2.54" y="99.06" drill="2"/>
+<hole x="2.54" y="2.54" drill="2.5"/>
+<hole x="246.38" y="99.06" drill="2.5"/>
+<hole x="246.38" y="2.54" drill="2.5"/>
+<hole x="2.54" y="99.06" drill="2.5"/>
 <wire x1="-5.08" y1="104.14" x2="-5.08" y2="-2.54" width="0" layer="48"/>
 <wire x1="-5.08" y1="-2.54" x2="-2.54" y2="-5.08" width="0" layer="48" curve="90"/>
@@
 <wire x1="126.365" y1="10.4775" x2="125.4125" y2="10.4775" width="2.0828" layer="25"/>
 <wire x1="125.095" y1="10.4775" x2="123.5075" y2="10.4775" width="2.0828" layer="25"/>
-<hole x="2.54" y="118.11" drill="2"/>
-<hole x="246.38" y="118.11" drill="2"/>
+<hole x="2.54" y="118.11" drill="2.5"/>
+<hole x="246.38" y="118.11" drill="2.5"/>
 <text x="208.385" y="1.27" size="3.302" layer="26" ratio="12" rot="MR0">A</text>
 <text x="204.575" y="1.27" size="1.27" layer="26" rot="MR0">Tip is +5V
@@
 Tom Armitage
 Brendan Cassidy</text>
-<text x="240.665" y="63.5" size="1.0668" layer="26" ratio="10" rot="MR0" align="top-left">v1.2</text>
+<text x="240.665" y="63.5" size="1.0668" layer="26" ratio="10" rot="MR0" align="top-left">v1.21</text>
 <text x="57.785" y="1.27" size="1.778" layer="25">I2C: Tip SDA, Ring SCL
 DO NOT HOT PLUG</text>
 <text x="243.205" y="21.9075" size="1.778" layer="25">MIDI</text>
 <text x="44.45" y="3.4925" size="1.778" layer="25" rot="R180">II</text>
+<hole x="63.5" y="63.5" drill="2.5"/>
+<hole x="185.42" y="63.5" drill="2.5"/>
+<hole x="124.46" y="63.5" drill="2.5"/>
 </plain>
 <attributes>
@@
 <attribute name="VALUE" x="47.3075" y="99.06" size="1.27" layer="27"/>
 </element>
-<element name="FID1" library="adafruit" library_urn="urn:adsk.eagle:library:420" package="FIDUCIAL_1MM" value="FIDUCIAL" x="2.54" y="115.57"/>
+<element name="FID1" library="adafruit" library_urn="urn:adsk.eagle:library:420" package="FIDUCIAL_1MM" value="FIDUCIAL" x="2.54" y="115"/>
 <element name="FID2" library="adafruit" library_urn="urn:adsk.eagle:library:420" package="FIDUCIAL_1MM" value="FIDUCIAL" x="246.38" y="6.35"/>
 <element name="JP2" library="SparkFun-Connectors" package="AUDIO-JACK" value="" x="50.4825" y="5.08" smashed="yes" rot="R90">
