File: electronics/16n_13.brd (EAGLE design)
At the start: 248.9 x 120.7 mm, 112 parts, among them J1 PJ302M, J10 PJ302M, J11 PJ302M, J12 PJ302M, J13 PJ302M, J14 PJ302M, J15 PJ302M, J16 PJ302M, J2 PJ302M, J3 PJ302M, J4 PJ302M, J5 PJ302M, J6 PJ302M, J7 PJ302M, J8 PJ302M, J9 PJ302M, U1 MCP6004_SMD, U2 MCP6004_SMD, U3 MCP6004_SMD, U4 MCP6004_SMD, U5 MCP6004_SMD, U6 MCP6004_SMD, U7 MCP6004_SMD, U8 MCP6004_SMD, U9 CD74HC4067SM96

Commit message: 1.31 board: updated component designators.
Parts:
- R1, R2: value 47 -> 1K
- R10, R14, R15, R5, R9: value 5.6K -> 1K
- R11, R13, R16, R6, R8: value 10K -> 1K
- R17: value 1K -> DNP
- R18: value 10K -> DNP
- R20, R24, R30, R34, R40, R44: value 5.6K -> 10K
- R21, R23, R31, R33, R41, R43: value 10K -> 5.6K
- R22, R32, R42, R46, R48, R51: value 1K -> 10K
- R27, R37, R45, R47, R50: value 1K -> 5.6K
- R3, R4: value DNP -> 1K
- R49, R52: value 1K -> 47
- U$1: value TEENSY_3.1-3.2_DIL -> SLIDEPOT-ALPS-60MM; device Teensy_3_and_LC_Series_Boards_v1.4:TEENSY_3.0-3.2&LC_DIL -> monome:RS6011SP600
- U$17: value SLIDEPOT-ALPS-60MM -> TEENSY_3.1-3.2_DIL; device monome:RS6011SP600 -> Teensy_3_and_LC_Series_Boards_v1.4:TEENSY_3.0-3.2&LC_DIL
- U1: value MCP6004_SMD -> CD74HC4067SM96; device MusicThingModular:SO14 -> foxfield:SOIC127P1030X265-24
- U9: value CD74HC4067SM96 -> MCP6004; device foxfield:SOIC127P1030X265-24 -> MusicThingModular:SO14
- moved R1 218.1 mm to (17.8, 101.6), turned to 0 degrees
- moved U$16 213.4 mm to (238.8, 63.5)
- moved U$2 213.4 mm to (25.4, 63.5)
- moved R2 203.1 mm to (33.0, 101.6), turned to 0 degrees
- moved R52 191.5 mm to (212.1, 2.54), turned to 180 degrees
- moved U$15 182.9 mm to (223.5, 63.5)
- moved U$3 182.9 mm to (40.6, 63.5)
- moved C9 167.7 mm to (231.1, 22.9), turned to 0 degrees
- moved U9 163.8 mm to (231.1, 16.5), turned to 270 degrees
- moved R45 158.6 mm to (195.3, 13.3), turned to 270 degrees
- moved U$14 152.4 mm to (208.3, 63.5)
- moved U$4 152.4 mm to (55.9, 63.5)
- moved R12 152.4 mm to (185.4, 101.6)
- moved R47 150.8 mm to (216.2, 13.3), turned to 270 degrees
- moved R16 136.0 mm to (245.1, 92.7), turned to 90 degrees
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Connections:
- net +3V3: now also C1.1, D1.C, R17.2, R18.2, R52.2, U$17.3.3V, U1.24; no longer C9.1, D2.C, R1.2, R3.2, R4.2, U$1.3.3V, U9.24
- net +5V: now also C9.1, U$1.1, U$17.VIN, U9.4; no longer C1.1, U$1.VIN, U$17.1, U1.4
- net A0: now also U1.9, U2.6, U2.7; no longer U1.6, U1.7, U9.9
- net A1: now also U2.8, U2.9; no longer U1.9, U9.8
- net A10: now also U1.18, U7.6, U7.7; no longer U6.6, U6.7, U9.18
- net A11: now also U1.19, U7.8, U7.9; no longer U6.8, U6.9, U9.19
- net A12: now also U1.20, U8.6, U8.7; no longer U7.6, U7.7, U9.20
- net A13: now also U1.21, U8.8, U8.9; no longer U7.8, U7.9, U9.21
- net A14: now also U1.22, U9.6, U9.7; no longer U8.6, U8.7, U9.22
- net A15: now also U1.23, U9.8, U9.9; no longer U8.8, U8.9, U9.23
- net A2: now also U1.7, U3.6, U3.7; no longer U2.6, U2.7, U9.7
- net A3: now also U1.6, U3.8, U3.9; no longer U2.8, U2.9, U9.6
- net A4: now also U1.5, U4.6, U4.7; no longer U3.6, U3.7, U9.5
- net A5: now also U1.4, U4.8, U4.9; no longer U3.8, U3.9, U9.4
- net A6: now also U1.3, U5.6, U5.7; no longer U4.6, U4.7, U9.3
- net A7: now also U1.2, U5.8, U5.9; no longer U4.8, U4.9, U9.2
- net A8: now also U1.16, U6.6, U6.7; no longer U5.6, U5.7, U9.16
- net A9: now also U1.17, U6.8, U6.9; no longer U5.8, U5.9, U9.17
- net ANALOG_IN: now also U$17.14/A0, U1.1; no longer U$1.14/A0, U9.1
- net CV1: now also R1.2; no longer R7.2
- net CV10: now also R10.2; no longer R48.2
- net CV11: now also R11.2; no longer R32.2
- net CV12: now also R12.2; no longer R49.2
- net CV13: now also R13.2; no longer R37.2
- net CV14: now also R14.2; no longer R50.2
- net CV15: now also R15.2; no longer R42.2
- net CV16: now also R16.2; no longer R51.2
- net CV2: now also R2.2; no longer R12.2
- net CV3: now also R3.2; no longer R52.2
- net CV4: now also R4.2; no longer R45.2
- net CV5: now also R5.2; no longer R17.2
- net CV6: now also R6.2; no longer R47.2
- net CV7: now also R7.2; no longer R22.2
- net CV8: now also R8.2; no longer R46.2
- net CV9: now also R9.2; no longer R27.2
- net GND: now also D2.A, R20.1, R22.1, R24.1, R30.1, R32.1, R34.1, R40.1, R42.1, R44.1, R46.1, R48.1, R51.1, U$1.3, U$17.AGND, U$17.GND, U1.12, U1.15, U9.11; no longer D1.A, R11.1, R13.1, R16.1, R18.1, R21.1, R23.1, R31.1, R33.1, R41.1, R43.1, R6.1, R8.1, U$1.AGND, U$1.GND, U$17.3, U1.11, U9.12, U9.15
- net MIDI_OUT: now also R49.2, U$17.1; no longer R2.2, U$1.1
- net N$10: now also R21.2, R22.2, U2.10; no longer R8.2, R9.2, U1.10
- net N$12: now also R39.2, R40.2, U4.5; no longer R15.2, R16.2, U3.5
- net N$13: now also R25.2, R26.2, U4.10; no longer R18.2, R19.2, U3.10
- net N$15: now also R41.2, R42.2, U5.5; no longer R20.2, R21.2, U4.5
- net N$16: now also R27.2, R28.2, U5.10; no longer R23.2, R24.2, U4.10
- net N$18: now also R43.2, R44.2, U6.5; no longer R25.2, R26.2, U5.5
- net N$19: now also R30.2, U6.10; no longer R28.2, U5.10
- net N$21: now also R45.2, R46.2, U7.5; no longer R30.2, R31.2, U6.5
- net N$22: now also R31.2, R32.2, U7.10; no longer R33.2, R34.2, U6.10
- net N$24: now also R47.2, R48.2, U8.5; no longer R35.2, R36.2, U7.5
- net N$25: now also R33.2, R34.2, U8.10; no longer R38.2, R39.2, U7.10
- net N$27: now also R50.2, R51.2, U9.5; no longer R40.2, R41.2, U8.5
- net N$28: now also R19.2, R20.2, U9.10; no longer R43.2, R44.2, U8.10
- net N$3: now also R49.1; no longer R2.1
- net N$300: now also R1.1, U2.1, U2.2; no longer R7.1, U1.1, U1.2
- net N$301: now also R2.1, U2.13, U2.14; no longer R12.1, U1.13, U1.14
- net N$302: now also R3.1, U3.1, U3.2; no longer R52.1, U2.1, U2.2
- net N$303: now also R4.1, U3.13, U3.14; no longer R45.1, U2.13, U2.14
- net N$304: now also R5.1, U4.1, U4.2; no longer R17.1, U3.1, U3.2
- net N$305: now also R6.1, U4.13, U4.14; no longer R47.1, U3.13, U3.14
- net N$306: now also R7.1, U5.1, U5.2; no longer R22.1, U4.1, U4.2
- net N$307: now also R8.1, U5.13, U5.14; no longer R46.1, U4.13, U4.14
- net N$308: now also R9.1, U6.1, U6.2; no longer R27.1, U5.1, U5.2
- net N$309: now also R10.1, U6.13, U6.14; no longer R48.1, U5.13, U5.14
- net N$310: now also R11.1, U7.1, U7.2; no longer R32.1, U6.1, U6.2
- net N$311: now also R12.1, U7.13, U7.14; no longer R49.1, U6.13, U6.14
- net N$312: now also R13.1, U8.1, U8.2; no longer R37.1, U7.1, U7.2
- net N$313: now also R14.1, U8.13, U8.14; no longer R50.1, U7.13, U7.14
- net N$314: now also R15.1, U9.1, U9.2; no longer R42.1, U8.1, U8.2
- net N$315: now also R16.1, U9.13, U9.14; no longer R51.1, U8.13, U8.14
- net N$4: now also R52.1; no longer R1.1
- net N$6: now also R37.2, R38.2, U3.5; no longer R10.2, R11.2, U2.5
- net N$7: now also R23.2, R24.2, U3.10; no longer R13.2, R14.2, U2.10
- net N$9: now also R35.2, R36.2, U2.5; no longer R5.2, R6.2, U1.5
- net S0: now also U$17.8, U1.10; no longer U$1.8, U9.10
- net S1: now also U$17.7, U1.11; no longer U$1.7, U9.11
- net S2: now also U$17.6, U1.14; no longer U$1.6, U9.14
- net S3: now also U$17.5, U1.13; no longer U$1.5, U9.13
- net SCL: now also D1.A, D2.C, R17.1, U$17.19/A5; no longer D3.C, D4.A, R4.1, U$1.19/A5
- net SDA: now also D3.C, D4.A, R18.1, U$17.18/A4; no longer D1.C, D2.A, R3.1, U$1.18/A4
- net W0: now also R35.1, U$1.2, U2.3; no longer R5.1, U$17.2, U1.3
- net W1: now also R21.1, U$2.2, U2.12; no longer R9.1, U$16.2, U1.12
- net W10: now also R45.1, U$11.2, U7.3; no longer R30.1, U$7.2, U6.3
- net W11: now also R31.1, U$12.2, U7.12; no longer R34.1, U$6.2, U6.12
- net W12: now also R47.1, U$13.2, U8.3; no longer R35.1, U$5.2, U7.3
- net W13: now also R33.1, U$14.2, U8.12; no longer R39.1, U$4.2, U7.12
- net W14: now also R50.1, U$15.2, U9.3; no longer R40.1, U$3.2, U8.3
- net W15: now also R19.1, U$16.2, U9.12; no longer R44.1, U$2.2, U8.12
- net W2: now also R37.1, U$3.2, U3.3; no longer R10.1, U$15.2, U2.3
- net W3: now also R23.1, U$4.2, U3.12; no longer R14.1, U$14.2, U2.12
- net W4: now also R39.1, U$5.2, U4.3; no longer R15.1, U$13.2, U3.3
- net W5: now also R25.1, U$6.2, U4.12; no longer R19.1, U$12.2, U3.12
- net W6: now also R41.1, U$7.2, U5.3; no longer R20.1, U$11.2, U4.3
- net W7: now also R27.1, U$8.2, U5.12; no longer R24.1, U$10.2, U4.12
- net W8: now also R43.1, U6.3; no longer R25.1, U5.3
- net W9: now also U$10.2, U6.12; no longer U$8.2, U5.12
Routing:
- net W0: track 156.3 -> 154.5 mm
- net W12: track 102.1 -> 100.9 mm
- net W8: track 117.2 -> 116.3 mm
