File: electronics/16n.sch (EAGLE design)
At the start: 112 parts, among them J1 PJ302M, J10 PJ302M, J11 PJ302M, J12 PJ302M, J13 PJ302M, J14 PJ302M, J15 PJ302M, J16 PJ302M, J2 PJ302M, J3 PJ302M, J4 PJ302M, J5 PJ302M, J6 PJ302M, J7 PJ302M, J8 PJ302M, J9 PJ302M, U1 CD74HC4067SM96, U2 MCP6004_SMD, U3 MCP6004_SMD, U4 MCP6004_SMD, U5 MCP6004_SMD, U6 MCP6004_SMD, U7 MCP6004_SMD, U8 MCP6004_SMD, U9 MCP6004

Commit message: Add frames and document versions to schematics, as per #4.
Other:
- moved on the sheet: C2, C3, C4, C5, C6, C7, C8, C9
